File: connectors.kicad_sch (KiCad schematic)
At the start: 6 parts, among them J1 0436500200, J2 0430450200, J3 TFM-115-02-S-D-WT, J4 TFM-115-02-S-D-WT, J5 0436500400, J7 0436500600

Commit message: PCB[Layout, Mounting]:Inital layout and edgecut/hole placment.
Parts:
- removed J5: 0436500400, remote_0436500400:CONN_SD-43650-001_04_MOL, symbol remote_0436500400:0436500400
- renumbered J2 to J1, J1 to J2, J7 to J5
Connections:
- net SDC_SENSE: now also J5.6; no longer J5.5
- net SDC_SENSE_RTN: now also J5.5; no longer J5.6
Other:
- moved on the sheet: J3, J4
