File: daisy_chain.kicad_sch (KiCad schematic)
At the start: 16 parts, among them U2 SM91502ALA-E, U3 SM91502ALA-E

Commit message: SCH[Pages, Chips]: Created page setup, and placed main IC's.
Parts:
- removed C1, C2, C3, C4: 220pF, remote_cl05a105ko5nnnc:C_0402_1005Metric, symbol remote_gcm1555c1h221ja16d:C
- removed CR1, CR2: PESD1CAN,215, remote_pesd1can_215:SOT23_PESD1_NEX, symbol remote_pesd1can_215:PESD1CAN_215
- added C11, C12, C13, C14: 100 pF, remote_cl05a105ko5nnnc:C_0402_1005Metric, symbol remote_gcm1555c1h101ja16d:C
- added D1, D2: PESD5V0U2BT-QR, remote_pesd5v0u2bt-qr:SOT-23-3, symbol remote_pesd5v0u2bt-qr:PESD5V0U2BT-QR
Connections:
- net COMH_WN: now also D1.2
- net COMH_WP: now also D1.1
- net COML_WN: now also D2.1
- net COML_WP: now also D2.2
- net GND: now also C11.1, C12.1, C13.1, C14.1, D1.3, D2.3
- net U1_COMH.N: now also C11.2
- net U1_COMH.P: now also C13.2
- net U1_COML.N: now also C14.2
- net U1_COML.P: now also C12.2

Commit message: SCH[Sens & Inputs, Logic]: Started on sens and inputs condtiong, Logic page drawn. Need to add notes still.
Changed lines of the file:
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@@
+		)
+	)
+	(hierarchical_label "COMH{P N}"
+		(shape bidirectional)
+		(at 307.34 78.74 0)
+		(effects
+			(font
+				(size 1.27 1.27)
+			)
+			(justify left)
+		)
+		(property "Netclass" "ISO"
+			(at 308.61 81.28 0)
+			(show_name no)
+			(do_not_autoplace no)
+			(effects
+				(font
+					(size 1.27 1.27)
+					(italic yes)
+				)
+				(justify left)
+			)
+		)
+	)
+	(hierarchical_label "COML{P N}"
+		(shape bidirectional)
+		(at 307.2245 127 0)
+		(effects
+			(font
+				(size 1.27 1.27)
+			)
+			(justify left)
+		)
+		(property "Netclass" "ISO"
+			(at 308.4945 129.54 0)
+			(show_name no)
+			(do_not_autoplace no)
+			(effects
+				(font
+					(size 1.27 1.27)
+					(italic yes)
+				)
+				(justify left)
+			)
 		)
 	)
@@
 			)
 		)
-	)
-	(hierarchical_label "COMH{P N}"
-		(shape bidirectional)
-		(at 307.34 78.74 0)
-		(effects
-			(font
-				(size 1.27 1.27)
-			)
-			(justify left)
-		)
-		(property "Netclass" "ISO"
-			(at 308.61 81.28 0)
-			(show_name no)
-			(do_not_autoplace no)
-			(effects
-				(font
-					(size 1.27 1.27)
-					(italic yes)
-				)
-				(justify left)
-			)
-		)
-	)
-	(hierarchical_label "COML{P N}"
-		(shape bidirectional)
-		(at 307.34 127 0)
-		(effects
-			(font
-				(size 1.27 1.27)
-			)
-			(justify left)
-		)
-		(property "Netclass" "ISO"
-			(at 308.61 129.54 0)
-			(show_name no)
-			(do_not_autoplace no)
-			(effects
-				(font
-					(size 1.27 1.27)
-					(italic yes)
-				)
-				(justify left)
-			)
-		)

Commit message: PCB[Layout, Mounting]:Inital layout and edgecut/hole placment.
Parts:
- renumbered C12 to C10, C13 to C5, C5 to C6, C11 to C7, C14 to C8, C6 to C9, R4 to R10, R5 to R11, R2 to R12, R6 to R13, R3 to R8, R1 to R9
Changed lines of the file:
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@@
 		(dnp no)
 		(fields_autoplaced yes)
-		(property "Reference" "C14"
+		(property "Reference" "C8"
 			(at 190.5 132.08 90)
 			(show_name no)
@@
 			(project "bms_master"
 				(path "/f9e05184-c88b-4a88-ae9c-ab2bdb32be7c/c5103ceb-5325-4a84-a025-9638a412984e/af224eec-27d8-4f88-a3c3-712d60217277"
-					(reference "C14")
+					(reference "C8")
 					(unit 1)
 				)
@@
 		(dnp no)
 		(fields_autoplaced yes)
-		(property "Reference" "C13"
+		(property "Reference" "C5"
 			(at 190.5 83.82 90)
 			(show_name no)
@@
 			(project "bms_master"
 				(path "/f9e05184-c88b-4a88-ae9c-ab2bdb32be7c/c5103ceb-5325-4a84-a025-9638a412984e/af224eec-27d8-4f88-a3c3-712d60217277"
-					(reference "C13")
+					(reference "C5")
 					(unit 1)
 				)
@@
 		(dnp no)
 		(fields_autoplaced yes)
-		(property "Reference" "#PWR053"
+		(property "Reference" "#PWR034"
 			(at 187.96 146.05 0)
 			(hide yes)
@@
 			(project "bms_master"
 				(path "/f9e05184-c88b-4a88-ae9c-ab2bdb32be7c/c5103ceb-5325-4a84-a025-9638a412984e/af224eec-27d8-4f88-a3c3-712d60217277"
-					(reference "#PWR053")
+					(reference "#PWR034")
 					(unit 1)
 				)
@@
 		(dnp no)
 		(fields_autoplaced yes)
-		(property "Reference" "#PWR054"
+		(property "Reference" "#PWR036"
 			(at 187.96 166.37 0)
 			(hide yes)
@@
 			(project "bms_master"
 				(path "/f9e05184-c88b-4a88-ae9c-ab2bdb32be7c/c5103ceb-5325-4a84-a025-9638a412984e/af224eec-27d8-4f88-a3c3-712d60217277"
-					(reference "#PWR054")
+					(reference "#PWR036")
 					(unit 1)
 				)
@@
 		(dnp no)
 		(fields_autoplaced yes)
-		(property "Reference" "#PWR056"
+		(property "Reference" "#PWR035"
 			(at 228.6 146.05 0)
 			(hide yes)
@@
 			(project "bms_master"
 				(path "/f9e05184-c88b-4a88-ae9c-ab2bdb32be7c/c5103ceb-5325-4a84-a025-9638a412984e/af224eec-27d8-4f88-a3c3-712d60217277"
-					(reference "#PWR056")
+					(reference "#PWR035")
 					(unit 1)
 				)
@@
 		(in_pos_files yes)
 		(dnp no)
-		(property "Reference" "R2"
+		(property "Reference" "R12"
 			(at 180.34 134.6199 90)
 			(show_name no)
@@
 			(project "bms_master"
 				(path "/f9e05184-c88b-4a88-ae9c-ab2bdb32be7c/c5103ceb-5325-4a84-a025-9638a412984e/af224eec-27d8-4f88-a3c3-712d60217277"
-					(reference "R2")
+					(reference "R12")
 					(unit 1)
 				)
@@
 		(in_pos_files yes)
 		(dnp no)
-		(property "Reference" "C5"
+		(property "Reference" "C6"
 			(at 234.95 85.09 0)
 			(show_name no)
@@
 			(project "bms_master"
 				(path "/f9e05184-c88b-4a88-ae9c-ab2bdb32be7c/c5103ceb-5325-4a84-a025-9638a412984e/af224eec-27d8-4f88-a3c3-712d60217277"
-					(reference "C5")
+					(reference "C6")
 					(unit 1)
 				)
@@
 		(dnp no)
 		(fields_autoplaced yes)
-		(property "Reference" "#PWR052"
+		(property "Reference" "#PWR033"
 			(at 187.96 118.11 0)
 			(hide yes)
@@
 			(project "bms_master"
 				(path "/f9e05184-c88b-4a88-ae9c-ab2bdb32be7c/c5103ceb-5325-4a84-a025-9638a412984e/af224eec-27d8-4f88-a3c3-712d60217277"
-					(reference "#PWR052")
+					(reference "#PWR033")
 					(unit 1)
 				)
@@
 		(in_pos_files yes)
 		(dnp no)
-		(property "Reference" "C6"
+		(property "Reference" "C9"
 			(at 234.95 133.35 0)
 			(show_name no)
@@
 			(project "bms_master"
 				(path "/f9e05184-c88b-4a88-ae9c-ab2bdb32be7c/c5103ceb-5325-4a84-a025-9638a412984e/af224eec-27d8-4f88-a3c3-712d60217277"
-					(reference "C6")
+					(reference "C9")
 					(unit 1)
 				)
@@
 		(dnp no)
 		(fields_autoplaced yes)
-		(property "Reference" "R6"
+		(property "Reference" "R13"
 			(at 199.39 140.97 0)
 			(show_name no)
@@
 			(project "bms_master"
 				(path "/f9e05184-c88b-4a88-ae9c-ab2bdb32be7c/c5103ceb-5325-4a84-a025-9638a412984e/af224eec-27d8-4f88-a3c3-712d60217277"
-					(reference "R6")
+					(reference "R13")
 					(unit 1)
 				)
@@
 		(dnp no)
 		(fields_autoplaced yes)
-		(property "Reference" "R3"
+		(property "Reference" "R8"
 			(at 199.39 72.39 0)
 			(show_name no)
@@
 			(project "bms_master"
 				(path "/f9e05184-c88b-4a88-ae9c-ab2bdb32be7c/c5103ceb-5325-4a84-a025-9638a412984e/af224eec-27d8-4f88-a3c3-712d60217277"
-					(reference "R3")
+					(reference "R8")
 					(unit 1)
 				)
@@
 		(dnp no)
 		(fields_autoplaced yes)
-		(property "Reference" "#PWR051"
+		(property "Reference" "#PWR031"
 			(at 187.96 97.79 0)
 			(hide yes)
@@
 			(project "bms_master"
 				(path "/f9e05184-c88b-4a88-ae9c-ab2bdb32be7c/c5103ceb-5325-4a84-a025-9638a412984e/af224eec-27d8-4f88-a3c3-712d60217277"
-					(reference "#PWR051")
+					(reference "#PWR031")
 					(unit 1)
 				)
@@
 		(in_pos_files yes)
 		(dnp no)
-		(property "Reference" "R1"
+		(property "Reference" "R9"
 			(at 180.34 86.3599 90)
 			(show_name no)
@@
 			(project "bms_master"
 				(path "/f9e05184-c88b-4a88-ae9c-ab2bdb32be7c/c5103ceb-5325-4a84-a025-9638a412984e/af224eec-27d8-4f88-a3c3-712d60217277"
-					(reference "R1")
+					(reference "R9")
 					(unit 1)
 				)
@@
 		(dnp no)
 		(fields_autoplaced yes)
-		(property "Reference" "C12"
+		(property "Reference" "C10"
 			(at 190.5 152.4 90)
 			(show_name no)
@@
 			(project "bms_master"
 				(path "/f9e05184-c88b-4a88-ae9c-ab2bdb32be7c/c5103ceb-5325-4a84-a025-9638a412984e/af224eec-27d8-4f88-a3c3-712d60217277"
-					(reference "C12")
+					(reference "C10")
 					(unit 1)
 				)
@@
 		(dnp no)
 		(fields_autoplaced yes)
-		(property "Reference" "#PWR055"
+		(property "Reference" "#PWR032"
 			(at 228.6 97.79 0)
 			(hide yes)
@@
 			(project "bms_master"
 				(path "/f9e05184-c88b-4a88-ae9c-ab2bdb32be7c/c5103ceb-5325-4a84-a025-9638a412984e/af224eec-27d8-4f88-a3c3-712d60217277"
-					(reference "#PWR055")
+					(reference "#PWR032")
 					(unit 1)
 				)
@@
 		(in_pos_files yes)
 		(dnp no)
-		(property "Reference" "#PWR049"
+		(property "Reference" "#PWR030"
 			(at 124.46 80.01 0)
 			(hide yes)
@@
 			(project "bms_master"
 				(path "/f9e05184-c88b-4a88-ae9c-ab2bdb32be7c/c5103ceb-5325-4a84-a025-9638a412984e/af224eec-27d8-4f88-a3c3-712d60217277"
-					(reference "#PWR049")
+					(reference "#PWR030")
 					(unit 1)
 				)
@@
 		(dnp no)
 		(fields_autoplaced yes)
-		(property "Reference" "R4"
+		(property "Reference" "R10"
 			(at 199.39 92.71 0)
 			(show_name no)
@@
 			(project "bms_master"
 				(path "/f9e05184-c88b-4a88-ae9c-ab2bdb32be7c/c5103ceb-5325-4a84-a025-9638a412984e/af224eec-27d8-4f88-a3c3-712d60217277"
-					(reference "R4")
+					(reference "R10")
 					(unit 1)
 				)
@@
 		(dnp no)
 		(fields_autoplaced yes)
-		(property "Reference" "C11"
+		(property "Reference" "C7"
 			(at 190.5 104.14 90)
 			(show_name no)
@@
 			(project "bms_master"
 				(path "/f9e05184-c88b-4a88-ae9c-ab2bdb32be7c/c5103ceb-5325-4a84-a025-9638a412984e/af224eec-27d8-4f88-a3c3-712d60217277"
-					(reference "C11")
+					(reference "C7")
 					(unit 1)
 				)
@@
 		(dnp no)
 		(fields_autoplaced yes)
-		(property "Reference" "R5"
+		(property "Reference" "R11"
 			(at 199.39 120.65 0)
 			(show_name no)
@@
 			(project "bms_master"
 				(path "/f9e05184-c88b-4a88-ae9c-ab2bdb32be7c/c5103ceb-5325-4a84-a025-9638a412984e/af224eec-27d8-4f88-a3c3-712d60217277"
-					(reference "R5")
+					(reference "R11")
 					(unit 1)
 				)
